File: board/smalltime.sch (KiCad schematic (older format))
At the start: 46 parts, among them IC1 STM32F030K6T6, IC2 DS3231MZ, IC3 ADP3338, J1 MICROUSB, P1 SWD, P2 SWD_TC, Q1 TEPT4400, Q2 Q_NMOS_GDS, Q3 Q_NMOS_GDS, Q4 Q_NMOS_GDS, Q5 Q_NMOS_GDS, Q6 Q_NMOS_GDS, Q7 Q_NMOS_GDS, Q8 Q_NMOS_GDS, Q9 Q_NMOS_GDS, SW1 INC, SW2 SET, U1 DIG1, U2 DIG2, U3 DIG3, U4 DIG4, U5 DIG5, U6 DIG6, U7 DIG7, U8 DIG8, X1 BATTERY

Commit message: Did some more routing.
Connections:
- net DIG1: now also IC1.25 (PA15)
- net DIG2: now also IC1.30 (PB7)
- net at IC1.26 (PB3): now also R5.2
- net at IC1.27 (PB4): now also R4.2
- net at IC1.28 (PB5): now also R9.2
- net at IC1.29 (PB6): now also R10.2
Other:
- moved on the sheet: P1, P2, R10, R4, R5, R9
Changed lines of the file:
@@
 LIBS:adp3338
 LIBS:smalltime-cache
-EELAYER 25 0
+EELAYER 26 0
 EELAYER END
 $Descr A4 11693 8268
@@
 L SWD_TC P2
 U 1 1 596FD9DC
-P 1300 4900
-F 0 "P2" H 1000 5100 50  0000 L CNN
-F 1 "SWD_TC" H 1000 4700 50  0000 L CNN
-F 2 "agg:TC2030-NL" H 1000 4600 50  0001 L CNN
-F 3 "" H 900 5000 50  0001 C CNN
-	1    1300 4900
+P 1250 5450
+F 0 "P2" H 950 5650 50  0000 L CNN
+F 1 "SWD_TC" H 950 5250 50  0000 L CNN
+F 2 "agg:TC2030-NL" H 950 5150 50  0001 L CNN
+F 3 "" H 850 5550 50  0001 C CNN
+	1    1250 5450
 	1    0    0    -1
 $EndComp
@@
 	0    1    1    0
 $EndComp
-Text Label 1800 4250 0    60   ~ 0
+Text Label 1750 4800 0    60   ~ 0
 ~RST
-Text Label 900  4900 2    60   ~ 0
+Text Label 850  5450 2    60   ~ 0
 ~RST
-Text Label 1800 3850 0    60   ~ 0
+Text Label 1750 4400 0    60   ~ 0
 SWDIO
-Text Label 1800 3950 0    60   ~ 0
+Text Label 1750 4500 0    60   ~ 0
 SWCLK
-Text Label 1700 4900 0    60   ~ 0
+Text Label 1650 5450 0    60   ~ 0
 SWCLK
-Text Label 1700 4800 0    60   ~ 0
+Text Label 1650 5350 0    60   ~ 0
 SWDIO
 Text Label 3450 3500 0    60   ~ 0
@@
 Text Label 4300 3700 0    60   ~ 0
 I2C_SCL
-NoConn ~ 1800 4050
-NoConn ~ 1800 4150
+NoConn ~ 1750 4600
+NoConn ~ 1750 4700
 $Comp
 L GND #PWR018
 U 1 1 59727F21
-P 750 4300
-F 0 "#PWR018" H 750 4050 50  0001 C CNN
-F 1 "GND" H 750 4150 50  0000 C CNN
-F 2 "" H 750 4300 50  0001 C CNN
-F 3 "" H 750 4300 50  0001 C CNN
-	1    750  4300
-	1    0    0    -1
-$EndComp
-Wire Wire Line
-	750  3950 750  4300
-Wire Wire Line
-	750  4250 800  4250
-Wire Wire Line
-	800  4050 750  4050
-Connection ~ 750  4250
-Wire Wire Line
-	800  3950 750  3950
-Connection ~ 750  4050
+P 700 4850
+F 0 "#PWR018" H 700 4600 50  0001 C CNN
+F 1 "GND" H 700 4700 50  0000 C CNN
+F 2 "" H 700 4850 50  0001 C CNN
+F 3 "" H 700 4850 50  0001 C CNN
+	1    700  4850
+	1    0    0    -1
+$EndComp
+Wire Wire Line
+	700  4500 700  4850
+Wire Wire Line
+	700  4800 750  4800
+Wire Wire Line
+	750  4600 700  4600
+Connection ~ 700  4800
+Wire Wire Line
+	750  4500 700  4500
+Connection ~ 700  4600
 $Comp
 L +3V3 #PWR019
 U 1 1 59727FB5
-P 750 3800
-F 0 "#PWR019" H 750 3650 50  0001 C CNN
-F 1 "+3V3" H 750 3940 50  0000 C CNN
-F 2 "" H 750 3800 50  0001 C CNN
-F 3 "" H 750 3800 50  0001 C CNN
-	1    750  3800
-	1    0    0    -1
-$EndComp
-Wire Wire Line
-	750  3850 800  3850
-Wire Wire Line
-	750  3800 750  3850
+P 700 4350
+F 0 "#PWR019" H 700 4200 50  0001 C CNN
+F 1 "+3V3" H 700 4490 50  0000 C CNN
+F 2 "" H 700 4350 50  0001 C CNN
+F 3 "" H 700 4350 50  0001 C CNN
+	1    700  4350
+	1    0    0    -1
+$EndComp
+Wire Wire Line
+	700  4400 750  4400
+Wire Wire Line
+	700  4350 700  4400
 $Comp
 L +3V3 #PWR020
 U 1 1 597280EE
-P 850 4750
-F 0 "#PWR020" H 850 4600 50  0001 C CNN
-F 1 "+3V3" H 850 4890 50  0000 C CNN
-F 2 "" H 850 4750 50  0001 C CNN
-F 3 "" H 850 4750 50  0001 C CNN
-	1    850  4750
-	1    0    0    -1
-$EndComp
-Wire Wire Line
-	850  4750 850  4800
-Wire Wire Line
-	850  4800 900  4800
+P 800 5300
+F 0 "#PWR020" H 800 5150 50  0001 C CNN
+F 1 "+3V3" H 800 5440 50  0000 C CNN
+F 2 "" H 800 5300 50  0001 C CNN
+F 3 "" H 800 5300 50  0001 C CNN
+	1    800  5300
+	1    0    0    -1
+$EndComp
+Wire Wire Line
+	800  5300 800  5350
+Wire Wire Line
+	800  5350 850  5350
 $Comp
 L GND #PWR021
 U 1 1 597281EA
-P 900 5000
-F 0 "#PWR021" H 900 4750 50  0001 C CNN
-F 1 "GND" H 900 4850 50  0000 C CNN
-F 2 "" H 900 5000 50  0001 C CNN
-F 3 "" H 900 5000 50  0001 C CNN
-	1    900  5000
-	1    0    0    -1
-$EndComp
-NoConn ~ 1700 5000
+P 850 5550
+F 0 "#PWR021" H 850 5300 50  0001 C CNN
+F 1 "GND" H 850 5400 50  0000 C CNN
+F 2 "" H 850 5550 50  0001 C CNN
+F 3 "" H 850 5550 50  0001 C CNN
+	1    850  5550
+	1    0    0    -1
+$EndComp
+NoConn ~ 1650 5550
 $Comp
 L +5V #PWR022
@@
 Text Label 6350 1350 2    60   ~ 0
 SEG_DP
-Text Label 4350 2450 0    60   ~ 0
+Text Label 2300 3800 2    60   ~ 0
 SEG_A
-Text Label 4350 2550 0    60   ~ 0
+Text Label 2300 3700 2    60   ~ 0
 SEG_B
 Text Label 4350 2650 0    60   ~ 0
@@
 Text Label 4350 2850 0    60   ~ 0
 SEG_E
-Text Label 4350 2950 0    60   ~ 0
+Text Label 2300 3900 2    60   ~ 0
 SEG_F
-Text Label 4350 3050 0    60   ~ 0
+Text Label 2300 4000 2    60   ~ 0
 SEG_G
 Text Label 4350 3150 0    60   ~ 0
 SEG_DP
-Text Label 4050 1500 0    60   ~ 0
+Text Label 3450 3700 0    60   ~ 0
 DIG1
-Text Label 4050 1600 0    60   ~ 0
+Text Label 2600 4200 2    60   ~ 0
 DIG2
 Text Label 4050 1700 0    60   ~ 0
@@
 L SWD P1
 U 1 1 596FD9A0
-P 1300 4050
-F 0 "P1" H 900 4350 50  0000 L CNN
-F 1 "SWD" H 900 3750 50  0000 L CNN
-F 2 "agg:FTSH-105-01-F-D-K" H 900 3650 50  0001 L CNN
-F 3 "" H 1650 3850 50  0001 C CNN
-F 4 "FTSH-105-01-F-D-K" H 900 3550 50  0001 L CNN "Toby"
-	1    1300 4050
+P 1250 4600
+F 0 "P1" H 850 4900 50  0000 L CNN
+F 1 "SWD" H 850 4300 50  0000 L CNN
+F 2 "agg:FTSH-105-01-F-D-K" H 850 4200 50  0001 L CNN
+F 3 "" H 1600 4400 50  0001 C CNN
+F 4 "FTSH-105-01-F-D-K" H 850 4100 50  0001 L CNN "Toby"
+	1    1250 4600
 	1    0    0    -1
 $EndComp
@@
 L R R4
 U 1 1 59799710
-P 4150 2450
-F 0 "R4" V 4100 2600 50  0000 C CNN
-F 1 "300" V 4150 2450 50  0000 C CNN
-F 2 "agg:0603" V 4080 2450 50  0001 C CNN
-F 3 "" H 4150 2450 50  0001 C CNN
-F 4 "2447331" H 4150 2450 60  0001 C CNN "Farnell"
-	1    4150 2450
-	0    1    1    0
-$EndComp
-Wire Wire Line
-	4300 2450 4350 2450
-Wire Wire Line
-	4300 2550 4350 2550
+P 2500 3800
+F 0 "R4" V 2450 3950 50  0000 C CNN
+F 1 "300" V 2500 3800 50  0000 C CNN
+F 2 "agg:0603" V 2430 3800 50  0001 C CNN
+F 3 "" H 2500 3800 50  0001 C CNN
+F 4 "2447331" H 2500 3800 60  0001 C CNN "Farnell"
+	1    2500 3800
+	0    -1   -1   0
+$EndComp
+Wire Wire Line
+	2350 3800 2300 3800
+Wire Wire Line
+	2350 3700 2300 3700
 Wire Wire Line
 	4300 2650 4350 2650
@@
 	4300 2850 4350 2850
 Wire Wire Line
-	4300 2950 4350 2950
-Wire Wire Line
-	4300 3050 4350 3050
+	2350 3900 2300 3900
+Wire Wire Line
+	2350 4000 2300 4000
 Wire Wire Line
 	4300 3150 4350 3150
@@
 L R R5
 U 1 1 59794DAB
-P 4150 2550
-F 0 "R5" V 4100 2700 50  0000 C CNN
-F 1 "300" V 4150 2550 50  0000 C CNN
-F 2 "agg:0603" V 4080 2550 50  0001 C CNN
-F 3 "" H 4150 2550 50  0001 C CNN
-F 4 "2447331" H 4150 2550 60  0001 C CNN "Farnell"
-	1    4150 2550
-	0    1    1    0
+P 2500 3700
+F 0 "R5" V 2450 3850 50  0000 C CNN
+F 1 "300" V 2500 3700 50  0000 C CNN
+F 2 "agg:0603" V 2430 3700 50  0001 C CNN
+F 3 "" H 2500 3700 50  0001 C CNN
+F 4 "2447331" H 2500 3700 60  0001 C CNN "Farnell"
+	1    2500 3700
+	0    -1   -1   0
 $EndComp
 $Comp
@@
 L R R9
 U 1 1 59794F04
-P 4150 2950
-F 0 "R9" V 4100 3100 50  0000 C CNN
-F 1 "300" V 4150 2950 50  0000 C CNN
-F 2 "agg:0603" V 4080 2950 50  0001 C CNN
-F 3 "" H 4150 2950 50  0001 C CNN
-F 4 "2447331" H 4150 2950 60  0001 C CNN "Farnell"
-	1    4150 2950
-	0    1    1    0
+P 2500 3900
+F 0 "R9" V 2450 4050 50  0000 C CNN
+F 1 "300" V 2500 3900 50  0000 C CNN
+F 2 "agg:0603" V 2430 3900 50  0001 C CNN
+F 3 "" H 2500 3900 50  0001 C CNN
+F 4 "2447331" H 2500 3900 60  0001 C CNN "Farnell"
+	1    2500 3900
+	0    -1   -1   0
 $EndComp
 $Comp
 L R R10
 U 1 1 59794F0B
-P 4150 3050
-F 0 "R10" V 4100 3200 50  0000 C CNN
-F 1 "300" V 4150 3050 50  0000 C CNN
-F 2 "agg:0603" V 4080 3050 50  0001 C CNN
-F 3 "" H 4150 3050 50  0001 C CNN
-F 4 "2447331" H 4150 3050 60  0001 C CNN "Farnell"
-	1    4150 3050
-	0    1    1    0
+P 2500 4000
+F 0 "R10" V 2450 4150 50  0000 C CNN
+F 1 "300" V 2500 4000 50  0000 C CNN
+F 2 "agg:0603" V 2430 4000 50  0001 C CNN
+F 3 "" H 2500 4000 50  0001 C CNN
+F 4 "2447331" H 2500 4000 60  0001 C CNN "Farnell"
+	1    2500 4000
+	0    -1   -1   0
 $EndComp
 $Comp
@@
 	3700 5950 3700 5650
 Connection ~ 3700 5650
+Wire Wire Line
+	2600 4200 2650 4200
+Wire Wire Line
+	2650 4200 2650 4100
 $EndSCHEMATC
